Commit message: adjusted urdf to dynamics model

File: planar_manipulator_defs/robots/planar_manipulator.urdf (robot description, URDF)
Before this commit: robot planar_manipulator, 9 links, 8 joints
Joints:
- joint 0_joint: origin xyz=0 0.05 0 rpy=0 0 0 -> xyz=0 0 0 rpy=0 0 0
- joint 1_joint: origin xyz=0 0.4 0 rpy=0 0 0 -> xyz=0.4 0 0 rpy=0 0 0
- joint 2_joint: origin xyz=0 0.4 0 rpy=0 0 0 -> xyz=0.4 0 0 rpy=0 0 0
- joint 3_joint: origin xyz=0 0.4 0 rpy=0 0 0 -> xyz=0.4 0 0 rpy=0 0 0
- joint 4_joint: origin xyz=0 0.4 0 rpy=0 0 0 -> xyz=0.4 0 0 rpy=0 0 0
- joint effector_joint: origin xyz=0 0.15 0 rpy=0 0 0 -> xyz=0.15 0 0 rpy=0 0 0
